File: kicad/C3I2.kicad_sch (KiCad schematic)
At the start: 37 parts, among them J1 1-84952-5, J2 PJRAN1X1U04X, J3 PJRAN1X1U04X, U1 ADV7280BCPZ-M-RL, U2 MIC5504-1.8YM5-TR, U3 MIC5504-1.8YM5-TR, Y1 28.63636MHz

Commit message: Revised PCB, issue 1
Parts:
- removed Y1: 28.63636MHz, components:XTAL_ABM8-28.63636MHZ-B2-T, symbol Device:Crystal
- added D2, D3, D4: LED, LED_SMD:LED_0805_2012Metric, symbol Device:LED
- added JP5: SolderJumper_3_Bridged12, Jumper:SolderJumper-3_P1.3mm_Bridged12_RoundedPad1.0x1.5mm_NumberLabels, symbol Jumper:SolderJumper_3_Bridged12
- added TP1, TP2: RCT-0C, digikey-footprints:PROBE_PAD_0805, symbol dk_Test-Points:RCT-0C
- added Y1: Crystal_GND24, components:XTAL_ABM8-28.63636MHZ-B2-T, symbol Device:Crystal_GND24
Connections:
- net +1V8: now also D2.2 (A); no longer R10.1, R9.1
- net +3.3V: now also R10.1, R9.1, D3.2 (A), JP5.2 (C)
- net GND: now also J2.1, J3.1, D2.1 (K), D3.1 (K), D4.1 (K), Y1.2, Y1.4; no longer J2.2, J2.3, J3.2, J3.3
- net I2C_SCL: now also TP2.1
- net I2C_SDA: now also TP1.1
- net PVDD: now also D4.2 (A)
- net PWR_EN: now also JP5.3 (B); no longer U2.3 (EN), U3.3 (EN)
- net at C2.2, U1.15 (XTALN): now also Y1.1
- net at C1.2, U1.14 (XTALP): now also Y1.3
- net at R3.1: now also J3.2, J3.3; no longer J3.1
- net at R1.1: now also J2.2, J2.3; no longer J2.1
- new net: JP5.1 (A), U2.3 (EN), U3.3 (EN)
Other:
- title: (none) -> C3I
- moved on the sheet: C1, C2, C3, C4, R1, R10, R2, R3, R4, R9
